File: hardware/pcb_module/dong_ho_module.kicad_sch (KiCad schematic)
At the start: 36 parts, among them J1 Motor rung 1027, J2 Pogo sạc (cái, nam châm), J3 Pin LiPo 603040 (JST PH2.0), J4 Dây sang BAT+/BAT- của XIAO, J5 Nút SOS, J6 Dây RA -> vít thép mép vỏ, Q1 AO3400A, U1 XIAO nRF52840 Sense, U2 MAX30102 (module tím), U3 CJMCU-30205, U4 AD8232 (module), U5 GC9A01 1.28in

Commit message: PCB module 1.1: dựng lại bằng KiCad 10 với MAX30102 2x4
- Chạy lại gen_fp/gen_sch/gen_pcb trên KiCad 10.0.7, thêm footprint Module_MAX30102_2x4.
- U2 đổi góc 180 -> 0 (vẫn lật mặt dưới) để chân khớp module thật:
  VIN (28,81; 24,92) ... INT (21,19; 35,08).
- D4 (TVS SMA) dời xuống y 35,4 để courtyard không chồng D5.
- Chữ chân U2 trên lụa 0,6/0,1 mm cho đúng quy tắc lụa.
- ERC 0 lỗi 0 cảnh báo; DRC 0 vi phạm, 0 chưa nối, khớp sơ đồ 0 lỗi.
- Xuất lại PDF, BOM, gerber + khoan, zip và ảnh 3D hai mặt.

Co-Authored-By: Claude Opus 5.5 <noreply@anthropic.com>
Claude-Session: https://claude.ai/code/session_016xjgaR8Q12uTCt4QMw8J44
Parts:
- removed D2, D3: 1N4148W, Diode_SMD:D_SOD-123, symbol Diode:1N4148W
- added D2, D3: 1N4148WS, Diode_SMD:D_SOD-323, symbol Diode:1N4148WS
- D4: value SMF5.0A -> SMAJ5.0A; footprint Diode_SMD:D_SOD-123F -> Diode_SMD:D_SMA; symbol Diode:SMF5V0A -> Diode:SMAJ5.0A
- U2: value MAX30102 (module tím) -> MAX30102 (module 2x4); footprint DoAnModule:Module_MAX30102_1x7 -> DoAnModule:Module_MAX30102_2x4
Connections:
- net ECG_LOD: now also D2.1 (K), D3.1 (K)
- net GND: now also U2.4 (GND), U2.5 (GND); no longer U2.7 (GND)
- net I2C_SCL: now also U2.3 (SCL); no longer U2.2 (SCL)
- net I2C_SDA: now also U2.2 (SDA); no longer U2.3 (SDA)
- net LO_N: now also D3.2 (A)
- net LO_P: now also D2.2 (A)
Other:
- note added: "Chân sạc pogo -> TVS SMAJ5.0A về GND -> SS14 nối tiếp -> chân 5V của XIAO. SS14 chặn dòng ngược từ USB-C ra chân pogo khi cắm cả hai. Mạch sạc LiPo nằm sẵn trên XIAO (BQ25101)."
- note added: "Module đen 2x4: VIN SDA SCL GND / GND RD IRD INT (đã đo 27/10/2026). INT, IRD, RD bỏ trống. Module có LDO 1,8 V và điện trở kéo lên riêng."
- note removed: "Chân sạc pogo -> TVS SMF5.0A về GND -> SS14 nối tiếp -> chân 5V của XIAO. SS14 chặn dòng ngược từ USB-C ra chân pogo khi cắm cả hai. Mạch sạc LiPo nằm sẵn trên XIAO (BQ25101)."
- note removed: "Thứ tự chân VIN SCL SDA INT IRD RD GND: kiểm tra trên module thật. INT, IRD, RD bỏ trống. Module có LDO 1,8 V và điện trở kéo lên riêng."
